Commit message: Added Gazebo launch file

File: description/robot_core.xacro (robot description, xacro)
@@ -41,4 +41,7 @@
     </xacro:inertial_box>
 </link>
+<gazebo reference="chassis">
+    <material>Gazebo/White</material>
+</gazebo>
 <!-- REAR LEFT WHEEL -->
 <joint name="rear_left_wheel_joint" type="continuous">
@@ -64,4 +67,7 @@
     </xacro:inertial_cylinder>
 </link>
+<gazebo reference="rear_left_wheel">
+    <material>Gazebo/Blue</material>
+</gazebo>
 <!-- REAR RIGHT WHEEL -->
 <joint name="rear_right_wheel_joint" type="continuous">
@@ -87,4 +93,7 @@
     </xacro:inertial_cylinder>
 </link>
+<gazebo reference="rear_right_wheel">
+    <material>Gazebo/Blue</material>
+</gazebo>
 <!-- FRONT RIGHT WHEEL -->
 <joint name="front_right_wheel_joint" type="continuous">
@@ -110,4 +119,7 @@
     </xacro:inertial_cylinder>
 </link>
+<gazebo reference="front_right_wheel">
+    <material>Gazebo/Blue</material>
+</gazebo>
 <!-- FRONT LEFT WHEEL -->
 <joint name="front_left_wheel_joint" type="continuous">
@@ -133,3 +145,6 @@
     </xacro:inertial_cylinder>
 </link>
+<gazebo reference="front_left_wheel">
+    <material>Gazebo/Blue</material>
+</gazebo>
 </robot>
