Commit message: Update ros2_control.xacro

File: description/ros2_control.xacro (robot description, xacro)
@@ -1,3 +1,46 @@
 <?xml version="1.0"?>
 <robot xmlns:xacro="http://www.ros.org/wiki/xacro"  name="robot">
+    <!-- tells gazebo the harware interface to load and which joints to asscoiate with -->
+    <ros2_control name="GazeboSystem" type="system">
+        <hardware>
+            <plugin>gazebo_ros2_control/GazeboSubsystem</plugin>
+        </hardware>
+        <joint name="front_left_wheel_joint">
+            <command_interface name = velocity>
+                <param name="min">-10</param>
+                <param name="max">10</param>
+            </command_interface>
+            <state_interface name="position" />
+            <state_interface name="velocity" />
+        <joint name="front_left_wheel_joint">
+        <joint name="back_left_wheel_joint">
+            <command_interface name = velocity>
+                <param name="min">-10</param>
+                <param name="max">10</param>
+            </command_interface>
+            <state_interface name="position" />
+            <state_interface name="velocity" />
+        <joint name="left_wheel_joint">
+        <joint name="front_right_wheel_joint">
+            <command_interface name = velocity>
+                <param name="min">-10</param>
+                <param name="max">10</param>
+            </command_interface>
+            <state_interface name="position" />
+            <state_interface name="velocity" />
+        <joint name="left_wheel_joint">
+        <joint name="back_right_wheel_joint">
+            <command_interface name = velocity>
+                <param name="min">-10</param>
+                <param name="max">10</param>
+            </command_interface>
+            <state_interface name="position" />
+            <state_interface name="velocity" />
+        <joint name="left_wheel_joint">
+    </ros2_control>
+    <gazebo>
+        <plugin filename="libgazebo_ros2_control.so" name="gazebo_ros2_control">
+            <!-- <parameters>...to be filled in soon!...</parameters> -->
+        </plugin>
+    </gazebo>
 </robot>

Commit message: updated joints in control

File: description/ros2_control.xacro (robot description, xacro)
@@ -13,5 +13,5 @@
             <state_interface name="position" />
             <state_interface name="velocity" />
-        <joint name="front_left_wheel_joint">
+        <joint>
         <joint name="back_left_wheel_joint">
             <command_interface name = velocity>
@@ -21,5 +21,5 @@
             <state_interface name="position" />
             <state_interface name="velocity" />
-        <joint name="left_wheel_joint">
+        <joint>
         <joint name="front_right_wheel_joint">
             <command_interface name = velocity>
@@ -29,5 +29,5 @@
             <state_interface name="position" />
             <state_interface name="velocity" />
-        <joint name="left_wheel_joint">
+        <joint>
         <joint name="back_right_wheel_joint">
             <command_interface name = velocity>
@@ -37,5 +37,5 @@
             <state_interface name="position" />
             <state_interface name="velocity" />
-        <joint name="left_wheel_joint">
+        <joint>
     </ros2_control>
     <gazebo>
